File: robocar-sensorbar/robocar-sensorbar.sch (KiCad schematic (older format))
At the start: 18 parts, among them J1 Conn_02x05_Odd_Even, U1 BPR-205, U2 BPR-205, U3 BPR-205, U4 BPR-205, U5 BPR-205

Commit message: 回路図の見栄えをよく
Parts:
- C1: value C -> 100n
- U1, U2, U3, U4, U5: value BPR-205 -> LBR-127HD
Changed lines of the file:
@@
 P 2200 2750
 F 0 "U1" H 2200 3067 50  0000 C CNN
-F 1 "BPR-205" H 2200 2976 50  0000 C CNN
+F 1 "LBR-127HD" H 2200 2976 50  0000 C CNN
 F 2 "photo-reflector:LBR-127HD" H 2200 2550 50  0001 C CNN
 F 3 "http://www.ystone.com.tw/en/data/goods/IRPT/Photo%20Interrupters-Reflective%20Type.pdf" H 2200 2850 50  0001 C CNN
@@
 P 4150 2750
 F 0 "U2" H 4150 3067 50  0000 C CNN
-F 1 "BPR-205" H 4150 2976 50  0000 C CNN
+F 1 "LBR-127HD" H 4150 2976 50  0000 C CNN
 F 2 "photo-reflector:LBR-127HD" H 4150 2550 50  0001 C CNN
 F 3 "http://www.ystone.com.tw/en/data/goods/IRPT/Photo%20Interrupters-Reflective%20Type.pdf" H 4150 2850 50  0001 C CNN
@@
 P 1800 4400
 F 0 "C1" H 1685 4354 50  0000 R CNN
-F 1 "C" H 1685 4445 50  0000 R CNN
+F 1 "100n" H 1685 4445 50  0000 R CNN
 F 2 "Capacitors_SMD:C_0603_HandSoldering" H 1838 4250 50  0001 C CNN
 F 3 "~" H 1800 4400 50  0001 C CNN
@@
 P 5600 2750
 F 0 "U3" H 5600 3067 50  0000 C CNN
-F 1 "BPR-205" H 5600 2976 50  0000 C CNN
+F 1 "LBR-127HD" H 5600 2976 50  0000 C CNN
 F 2 "photo-reflector:LBR-127HD" H 5600 2550 50  0001 C CNN
 F 3 "http://www.ystone.com.tw/en/data/goods/IRPT/Photo%20Interrupters-Reflective%20Type.pdf" H 5600 2850 50  0001 C CNN
@@
 P 7100 2750
 F 0 "U4" H 7100 3067 50  0000 C CNN
-F 1 "BPR-205" H 7100 2976 50  0000 C CNN
+F 1 "LBR-127HD" H 7100 2976 50  0000 C CNN
 F 2 "photo-reflector:LBR-127HD" H 7100 2550 50  0001 C CNN
 F 3 "http://www.ystone.com.tw/en/data/goods/IRPT/Photo%20Interrupters-Reflective%20Type.pdf" H 7100 2850 50  0001 C CNN
@@
 P 8650 2750
 F 0 "U5" H 8650 3067 50  0000 C CNN
-F 1 "BPR-205" H 8650 2976 50  0000 C CNN
+F 1 "LBR-127HD" H 8650 2976 50  0000 C CNN
 F 2 "photo-reflector:LBR-127HD" H 8650 2550 50  0001 C CNN
 F 3 "http://www.ystone.com.tw/en/data/goods/IRPT/Photo%20Interrupters-Reflective%20Type.pdf" H 8650 2850 50  0001 C CNN
