File: robocar-mainboard/robocar-mainboard.sch (KiCad schematic (older format))
At the start: 37 parts, among them J1 PSEL, J2 Batt1, J3 USB_B, J4 JTAG, J5 SensorBoard, J6 Batt2, J7 MotorL, J8 MotorR, Q1 2SC2712, Q2 2SC2712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

Commit message: 回路図の見栄えをよく
Parts:
- D1: value LED -> LED_RED
- D2: value LED -> LED_GREEN
- D3: value LED -> LED_YELLOW
- R2, R3: value 10k -> 330
- R4: value R -> 470
- U4: symbol Akizuki-Kit:AE-DRV8835-S -> robocar-mainboard-rescue:AE-DRV8835-S-Akizuki-Kit
Connections:
- net SW_USER: now reaches C8.1, SW3.1, U2.30 (IO18)
- no-connect marks 0 -> 10
Other:
- note added: "Connectors"
- note added: "ESP32"
- note added: "Motor Driver"
- note added: "Power"
- note added: "USB & Programming"
- moved on the sheet: C1, C2, C3, C4, C5, C6, C7, C8, D1, D2, D3, J1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

Commit message: 諸々整理
Parts:
- U4: symbol robocar-mainboard-rescue:AE-DRV8835-S-Akizuki-Kit -> Akizuki-Kit:AE-DRV8835-S
Changed lines of the file:
@@
 EESchema Schematic File Version 4
 LIBS:robocar-mainboard-cache
-EELAYER 26 0
+EELAYER 30 0
 EELAYER END
 $Descr A4 11693 8268
@@
 Motor Battery
 $Comp
-L robocar-mainboard-rescue:AE-DRV8835-S-Akizuki-Kit U4
+L Akizuki-Kit:AE-DRV8835-S U4
 U 1 1 5D57410D
 P 2500 6650
